File: pcb/demo.kicad_pcb (KiCad board)
At the start: 2 copper layers, 41.9 x 25.4 mm, 18 parts, among them J1 Conn_01x01_Pin, J2 Conn_01x01_Pin, Q1 BC547, Q2 BC547

Commit message: Update to KiCAD 9
Parts:
- Q1, Q2: footprint Package_TO_SOT_THT:TO-92_Inline_Wide -> Package_TO_SOT_THT:TO-92L_Inline_Wide
Other:
- outline, holes or cut-outs redrawn
