File: pcb/demo.kicad_sch (KiCad schematic)
At the start: 18 parts, among them J1 Conn_01x01_Pin, J2 Conn_01x01_Pin, Q1 BC547, Q2 BC547

Commit message: Update to KiCAD 9
Parts:
- removed Q1, Q2: BC547, Package_TO_SOT_THT:TO-92_Inline_Wide, symbol Device:Q_NPN_CBE
- added Q1, Q2: BC547, Package_TO_SOT_THT:TO-92L_Inline_Wide, symbol Transistor_BJT:BC547
- FID1, FID2, FID3, FID4, H1, H2: now left out of the parts list
Connections:
- net GND: now also Q1.3 (E), Q2.3 (E)
- net at C2.1, R2.2: now also Q2.1 (C)
- net at C2.2, R4.2: now also Q1.2 (B)
- net at C1.1, R1.2: now also Q1.1 (C)
- net at C1.2, R3.2: now also Q2.2 (B)
