File: pcb/demo.kicad_sch (KiCad schematic)
At the start: 18 parts, among them J1 Conn_01x01_Pin, J2 Conn_01x01_Pin, Q1 BC547, Q2 BC547

Commit message: Rename/Add/Remove bom fields
Parts:
- C1, C2: HTL (none) -> 100354; Vendor HTL -> (none); VendorId 100354 -> (none)
- D1, D2: HTL (none) -> 100445, 100444; Vendor HTL -> (none); VendorId 100445, 100444 -> (none)
- H1, H2: HTL (none) -> 101017, 101382; Vendor HTL -> (none); VendorId 101017, 101382 -> (none)
- J1, J2: HTL (none) -> 101521; Vendor HTL -> (none); VendorId 101521 -> (none)
- Q1, Q2: HTL (none) -> 100215; Vendor HTL -> (none); VendorId 100215 -> (none)
- R1, R2: HTL (none) -> 102800; Vendor HTL -> (none); VendorId 102800 -> (none)
- R3, R4: HTL (none) -> 102812; Vendor HTL -> (none); VendorId 102812 -> (none)
Changed lines of the file:
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@@
 			)
 		)
-		(property "Vendor" "HTL"
-			(at 177.8 95.25 0)
-			(effects
-				(font
-					(size 1.27 1.27)
-				)
-				(hide yes)
-			)
-		)
-		(property "VendorId" "102800"
+		(property "HTL" "102800"
 			(at 177.8 95.25 0)
 			(effects
@@
 			)
 		)
-		(property "Vendor" "HTL"
-			(at 175.26 114.3 0)
-			(effects
-				(font
-					(size 1.27 1.27)
-				)
-				(hide yes)
-			)
-		)
-		(property "VendorId" "100215"
+		(property "HTL" "100215"
 			(at 175.26 114.3 0)
 			(effects
@@
 			)
 		)
-		(property "Vendor" ""
-			(at 38.1 165.1 0)
-			(effects
-				(font
-					(size 1.27 1.27)
-				)
-				(hide yes)
-			)
-		)
-		(property "VendorId" ""
-			(at 38.1 165.1 0)
-			(effects
-				(font
-					(size 1.27 1.27)
-				)
-				(hide yes)
-			)
-		)
 		(instances
 			(project "demo"
@@
 					(size 1.27 1.27)
 				)
-			)
-		)
-		(property "Vendor" ""
-			(at 50.8 165.1 0)
-			(effects
-				(font
-					(size 1.27 1.27)
-				)
-				(hide yes)
-			)
-		)
-		(property "VendorId" ""
-			(at 50.8 165.1 0)
-			(effects
-				(font
-					(size 1.27 1.27)
-				)
-				(hide yes)
 			)
 		)
@@
 			)
 		)
-		(property "Vendor" "HTL"
-			(at 158.75 88.9 0)
-			(effects
-				(font
-					(size 1.27 1.27)
-				)
-				(hide yes)
-			)
-		)
-		(property "VendorId" "102812"
+		(property "HTL" "102812"
 			(at 158.75 88.9 0)
 			(effects
@@
 			)
 		)
-		(property "Vendor" "HTL"
-			(at 177.8 82.55 0)
-			(effects
-				(font
-					(size 1.27 1.27)
-				)
-				(hide yes)
-			)
-		)
-		(property "VendorId" "100445, 100444"
-			(at 177.8 82.55 0)
-			(effects
-				(font
-					(size 1.27 1.27)
-				)
-				(hide yes)
-			)
-		)
 		(property "Sim.Pins" "1=K 2=A"
 			(at 177.8 82.55 0)
+			(effects
+				(font
+					(size 1.27 1.27)
+				)
+				(hide yes)
+			)
+		)
+		(property "HTL" "100445, 100444"
+			(at 177.8 82.55 90)
 			(effects
 				(font
@@
 			)
 		)
-		(property "Vendor" "HTL"
-			(at 165.1 104.14 0)
-			(effects
-				(font
-					(size 1.27 1.27)
-				)
-				(hide yes)
-			)
-		)
-		(property "VendorId" "100354"
-			(at 165.1 104.14 0)
+		(property "HTL" "100354"
+			(at 165.1 104.14 90)
 			(effects
 				(font
@@
 			)
 		)
-		(property "Vendor" "HTL"
-			(at 109.22 121.92 0)
-			(effects
-				(font
-					(size 1.27 1.27)
-				)
-				(hide yes)
-			)
-		)
-		(property "VendorId" "101521"
+		(property "HTL" "101521"
 			(at 109.22 121.92 0)
 			(effects
@@
 			)
 		)
-		(property "Vendor" "HTL"
-			(at 146.05 88.9 0)
-			(effects
-				(font
-					(size 1.27 1.27)
-				)
-				(hide yes)
-			)
-		)
-		(property "VendorId" "102812"
+		(property "HTL" "102812"
 			(at 146.05 88.9 0)
 			(effects
@@
 			)
 		)
-		(property "Vendor" "HTL"
-			(at 139.7 104.14 0)
-			(effects
-				(font
-					(size 1.27 1.27)
-				)
-				(hide yes)
-			)
-		)
-		(property "VendorId" "100354"
-			(at 139.7 104.14 0)
+		(property "HTL" "100354"
+			(at 139.7 104.14 90)
 			(effects
 				(font
@@
 			)
 		)
-		(property "Vendor" "HTL"
-			(at 114.3 166.37 0)
-			(effects
-				(font
-					(size 1.27 1.27)
-				)
-				(hide yes)
-			)
-		)
-		(property "VendorId" "101017, 101382"
-			(at 114.3 166.37 0)
+		(property "HTL" "101017, 101382"
+			(at 114.3 166.37 90)
 			(effects
 				(font
@@
 			)
 		)
-		(property "Vendor" "HTL"
-			(at 101.6 166.37 0)
-			(effects
-				(font
-					(size 1.27 1.27)
-				)
-				(hide yes)
-			)
-		)
-		(property "VendorId" "101017, 101382"
-			(at 101.6 166.37 0)
+		(property "HTL" "101017, 101382"
+			(at 101.6 166.37 90)
 			(effects
 				(font
@@
 			)
 		)
-		(property "Vendor" "HTL"
-			(at 109.22 76.2 0)
-			(effects
-				(font
-					(size 1.27 1.27)
-				)
-				(hide yes)
-			)
-		)
-		(property "VendorId" "101521"
+		(property "HTL" "101521"
 			(at 109.22 76.2 0)
 			(effects
@@
 			)
 		)
-		(property "Vendor" "HTL"
-			(at 127 82.55 0)
-			(effects
-				(font
-					(size 1.27 1.27)
-				)
-				(hide yes)
-			)
-		)
-		(property "VendorId" "100445, 100444"
-			(at 127 82.55 0)
-			(effects
-				(font
-					(size 1.27 1.27)
-				)
-				(hide yes)
-			)
-		)
 		(property "Sim.Pins" "1=K 2=A"
 			(at 127 82.55 0)
@@
 			)
 		)
+		(property "HTL" "100445, 100444"
+			(at 127 82.55 90)
+			(effects
+				(font
+					(size 1.27 1.27)
+				)
+				(hide yes)
+			)
+		)
 		(pin "1"
 		)
@@
 					(size 1.27 1.27)
 				)
-			)
-		)
-		(property "Vendor" ""
-			(at 76.2 165.1 0)
-			(effects
-				(font
-					(size 1.27 1.27)
-				)
-				(hide yes)
-			)
-		)
-		(property "VendorId" ""
-			(at 76.2 165.1 0)
-			(effects
-				(font
-					(size 1.27 1.27)
-				)
-				(hide yes)
 			)
 		)
@@
 			)
 		)
-		(property "Vendor" "HTL"
-			(at 129.54 114.3 0)
-			(effects
-				(font
-					(size 1.27 1.27)
-				)
-				(hide yes)
-			)
-		)
-		(property "VendorId" "100215"
+		(property "HTL" "100215"
 			(at 129.54 114.3 0)
 			(effects
@@
 					(size 1.27 1.27)
 				)
-			)
-		)
-		(property "Vendor" ""
-			(at 63.5 165.1 0)
-			(effects
-				(font
-					(size 1.27 1.27)
-				)
-				(hide yes)
-			)
-		)
-		(property "VendorId" ""
-			(at 63.5 165.1 0)
-			(effects
-				(font
-					(size 1.27 1.27)
-				)
-				(hide yes)
 			)
 		)
@@
 			)
 		)
-		(property "Vendor" "HTL"
+		(property "HTL" "102800"
 			(at 127 95.25 0)
 			(effects
-				(font
-					(size 1.27 1.27)
-				)
-				(hide yes)
-			)
-		)
-		(property "VendorId" "102800"
-			(at 127 95.25 0)
-			(effects
